File: PandoPad/PandoPad.kicad_sch (KiCad schematic)
At the start: 90 parts, among them J1 78171-0004, J2 Conn_01x05, J3 MalePogo, J4 FemalePogo, K1 Num, K10 8, K11 9, K12 Right+, K13 4, K14 5, K15 6, K16 OPT2, K17 1, K18 2, K19 3, K2 /, K20 REnt, K22 LZero, K23 ., K24 ., K25 OPT5, K3 *, K4 -, K9 7, P1 OLED1, P2 OLED2, P3 OLED2, SW1 Mod1, SW1 SW_Push, SW2 Mod2, SW3 Mod3, SW4 Mod4, U1 W25Q128JVS, U3 RP2040, U4 XC6206PxxxMR-Regulator_Linear, Y1 12MHz

Commit message: Finished Routing
Parts:
- removed K1: Num, Switch_Keyboard_Hotswap_Kailh:SW_Hotswap_Kailh_MX_plated_1.00u_Vias, symbol Switch:SW_Push
- removed K2: /, Switch_Keyboard_Hotswap_Kailh:SW_Hotswap_Kailh_MX_plated_1.00u_Vias, symbol Switch:SW_Push
- removed K3: *, Switch_Keyboard_Hotswap_Kailh:SW_Hotswap_Kailh_MX_plated_1.00u_Vias, symbol Switch:SW_Push
- removed K4: -, Switch_Keyboard_Hotswap_Kailh:SW_Hotswap_Kailh_MX_plated_1.00u_Vias, symbol Switch:SW_Push
- removed P1: OLED1, Libraries:OLED_v2, symbol Connector:Conn_01x04_Male
- removed P2: OLED2, Libraries:OLED_v2, symbol Connector:Conn_01x04_Male
- removed SW1: Mod1, Switch_Keyboard_Hotswap_Kailh:SW_Hotswap_Kailh_MX_plated_1.00u_Enc_Standalone, symbol marbastlib-various:Hotswap_MX_Encoder
- removed SW2: Mod2, Switch_Keyboard_Hotswap_Kailh:SW_Hotswap_Kailh_MX_plated_1.00u_Enc_Standalone, symbol marbastlib-various:Hotswap_MX_Encoder
- removed SW3: Mod3, Switch_Keyboard_Hotswap_Kailh:SW_Hotswap_Kailh_MX_plated_1.00u_Enc_Standalone, symbol marbastlib-various:Hotswap_MX_Encoder
- removed SW4: Mod4, Switch_Keyboard_Hotswap_Kailh:SW_Hotswap_Kailh_MX_plated_1.00u_Enc_Standalone, symbol marbastlib-various:Hotswap_MX_Encoder
- removed U1: W25Q128JVS, Package_SO:SOIC-8_5.23x5.23mm_P1.27mm, symbol Memory_Flash:W25Q128JVS
- added K1, K2, K3, K4: ~, Switch_Keyboard_Hotswap_Kailh:SW_Hotswap_Kailh_MX_plated_1.00u_Enc_Standalone, symbol skyloong:SKYLOONG
- added Q1, Q2, Q3, Q4: PMOS, Keebio-Parts:SOT-23, symbol Simulation_SPICE:PMOS
- added R6, R7, R8, R9: 1k, Resistor_SMD:R_0603_1608Metric, symbol Device:R
- added U4: W25Q32JVUUIQ, Extra-components:SON80P400X300X60-10N, symbol USON-8(4x3):AT25SL321-MBUE-T
- J2: footprint Connector_PinSocket_2.54mm:PinSocket_1x05_P2.54mm_Vertical -> Connector_PinHeader_2.00mm:PinHeader_1x05_P2.00mm_Vertical
- J3: footprint Connector_PinHeader_2.54mm:PinHeader_1x04_P2.54mm_Vertical -> Extra-components:1x04_3.00mm_Magnetic Pogo_Male
- J4: footprint Connector_PinHeader_2.54mm:PinHeader_1x04_P2.54mm_Vertical -> Extra-components:1x04_3.00mm_Magnetic Pogo_Female
- R1, R2, R7: footprint Resistor_SMD:R_0402_1005Metric -> Resistor_SMD:R_0603_1608Metric
- SW1: footprint Keebio-Parts:SW_SPST_TL3342 -> marbastlib-various:SW_C843666
- renumbered P3 to P1
Connections:
- net GPIO0 is gone; now on net E2A: U3.2 (GPIO0)
- net GPIO1 is gone; now on net E2B: U3.3 (GPIO1)
- net GPIO10 is gone; now on net row4: U3.13 (GPIO10)
- net GPIO11 is gone; now on net row3: U3.14 (GPIO11)
- net GPIO14 is gone; now on net col1: U3.17 (GPIO14)
- net GPIO18 is gone; now on net row2: U3.29 (GPIO18)
- net GPIO19 is gone; now on net col0: U3.30 (GPIO19)
- net GPIO2 is gone; now on net E3A: U3.4 (GPIO2)
- net GPIO20 is gone; now on net row0: U3.31 (GPIO20)
- net GPIO22 is gone; now on net E1A: U3.34 (GPIO22)
- net GPIO23 is gone; now on net E1B: U3.35 (GPIO23)
- net GPIO3 is gone; now on net E3B: U3.5 (GPIO3)
- net GPIO4 is gone; now on net E4B: U3.6 (GPIO4)
- net GPIO5 is gone; now on net E4A: U3.7 (GPIO5)
- net GPIO6 is gone; now on net col3: U3.8 (GPIO6)
- net GPIO7 is gone; now on net col2: U3.9 (GPIO7)
- net row5 is gone; now on net row4: D21.1 (K), D22.1 (K), D23.1 (K), D24.1 (K)
- net +3V3: now also J2.1 (Pin_1), J3.1 (Pin_1), J4.1 (Pin_1), R6.1, R7.1, R8.1, R9.1, U4.8 (VCC); no longer J2.2 (Pin_2), J3.4 (Pin_4), J4.4 (Pin_4)
- net CS: now also U4.1 (~{CS})
- net E1A: now also K1.A
- net E1B: now also K1.B
- net E2A: now also K2.A
- net E2B: now also K2.B
- net E3A: now also K3.A
- net E3B: now also K3.B
- net E4A: now also K4.A
- net E4B: now also K4.B
- net GND: now also J2.5 (Pin_5), J3.4 (Pin_4), J4.4 (Pin_4), K1.C, K2.C, K3.C, K4.C, U4.10 (EXP), U4.4 (GND), U4.9 (EXP); no longer J2.3 (Pin_3), J3.1 (Pin_1), J4.1 (Pin_1)
- net QSPI_CLK: now also U4.6 (SCK)
- net SD0: now also U4.5 (SI(I/O0))
- net SD1: now also U4.2 (SO(I/O1))
- net SD2: now also U4.3 (~{WP~{(I/O2)})
- net SD3: now also U4.7 (~{HOLD~{/~{RESET~{(I/O3)})
- net SWCLK: now also J2.2 (Pin_2); no longer J2.5 (Pin_5)
- net SWD: now also J2.3 (Pin_3); no longer J2.4 (Pin_4)
- net XTAL_IN: now also Y1.1; no longer Y1.3
- net XTAL_O: now also Y1.3; no longer Y1.1
- net col0: now also K13.2, K17.2, K22.2, K9.2, KO-1.2, KO-3.2, KO-5.2, K1.1, Q1.1 (D)
- net col1: now also K10.2, K14.2, K18.2, K23.2, K2.1, Q2.1 (D)
- net col2: now also K11.2, K15.2, K19.2, K24.2, K3.1, Q3.1 (D)
- net col3: now also K12.2, K16.2, K20.2, K25.2, KO-2.2, KO-4.2, KO-6.2, K4.1, Q4.1 (D)
- net row2: now also D13.1 (K), D14.1 (K), D15.1 (K), D16.1 (K); no longer D10.1 (K), D11.1 (K), D12.1 (K), D9.1 (K)
- net row3: now also D17.1 (K), D18.1 (K), D19.1 (K), D20.1 (K); no longer D13.1 (K), D14.1 (K), D15.1 (K), D16.1 (K)
- net row4: no longer D17.1 (K), D18.1 (K), D19.1 (K), D20.1 (K)
- net ~{RESET}: now also J2.4 (Pin_4); no longer J2.1 (Pin_1)
- net at D2.2 (A): now also K2.2, Q2.3 (S)
- net at D3.2 (A): now also K3.2, Q3.3 (S)
- net at D1.2 (A): now also K1.2, Q1.3 (S)
- net at D4.2 (A): now also K4.2, Q4.3 (S)
- net GPIO12: no longer names the net of U3.15 (GPIO12)
- net GPIO13: no longer names the net of U3.16 (GPIO13)
- net GPIO15: no longer names the net of U3.18 (GPIO15)
- net GPIO16: no longer names the net of U3.27 (GPIO16)
- net GPIO17: no longer names the net of U3.28 (GPIO17)
- net GPIO21 renamed row1
- net row1: now also D10.1 (K), D11.1 (K), D12.1 (K), D9.1 (K)
- net GPIO24: no longer names the net of U3.36 (GPIO24)
- net GPIO25: no longer names the net of U3.37 (GPIO25)
- net GPIO26: no longer names the net of U3.38 (GPIO26/ADC0)
- net GPIO27: no longer names the net of U3.39 (GPIO27/ADC1)
- net GPIO28: no longer names the net of U3.40 (GPIO28/ADC2)
- net GPIO29: no longer names the net of U3.41 (GPIO29/ADC3)
- net GPIO8: no longer names the net of U3.11 (GPIO8)
- net GPIO9: no longer names the net of U3.12 (GPIO9)
- new net: K1.S, Q1.2 (G), R6.2
- new net: K2.S, Q2.2 (G), R7.2
- new net: K4.S, Q4.2 (G), R9.2
- new net: K3.S, Q3.2 (G), R8.2
Other:
- moved on the sheet: C10, C11, C12, C13, C14, C15, C16, C17, C2, C3, C4, C5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
